Commit message: wrong link name  in urdf

File: automatica2014_description/urdf/sia10f.urdf.xacro (robot description, xacro)
@@ -1,2 +1,3 @@
+<?xml version="1.0"?>
     <robot xmlns:xacro="http://ros.org/wiki/xacro" name="sia10f">
                 <xacro:property name="gripper_origin">
@@ -21,5 +22,5 @@
                 <!-- gripper -->
                 <joint name="flange_joint" type="fixed" >
-                    <parent link="sia10f_link_7_t" />
+                    <parent link="sia10f_link_t" />
                     <child link="gripper_flange_link" />
                     <xacro:insert_block name="flange_origin" />
